File: linkitsmart7688duo_doorcontroller.sch (EAGLE design)
At the start: 52 parts, among them CN1 4p-2.54-h8.5, CN2 4p-2.54-h8.5, J1 20p-2.54, J4 20p-2.54, J7 320140010, U2 RS485SOIC

Commit message: labeled stuff in schematic
Other:
- note added: "Ethernet"
- note added: "Linkit Smart 7688 DUO"
- note added: "RS485 - Jumper pins to move between UART0 and UART1"
- note added: "Silly RGB LEDs"
- note added: "Switched Ground for Door Mosfet Maglock, Ground supply and VRAW for motion detectos and Maglock, Optocoupler for 12v sensing input of door state"
- note removed: "RS485"
- moved on the sheet: CN1, CN2, D1, J1, J2, J3, J4, OC1, OC2, Q1, Q2, Q3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
